File: LEDboard.kicad_pcb (KiCad board)
At the start: 2 copper layers, 70 x 30 mm, 12 parts, among them J1 Conn_01x03, J2 Conn_01x03

Commit message: KiCad8.0にアップデート
Parts:
- J1, J2: footprint my_parts_lib:EuroBlock_receptacle_2.54_3p -> SamacSys_Parts:EuroBlock_receptacle_2.54_3p
