File: LEDboard.kicad_sch (KiCad schematic)
At the start: 12 parts, among them J1 Conn_01x03, J2 Conn_01x03

Commit message: KiCad8.0にアップデート
Parts:
- J1, J2: footprint my_parts_lib:EuroBlock_receptacle_2.54_3p -> SamacSys_Parts:EuroBlock_receptacle_2.54_3p
